File: without-power-switch-percent-mod/u1_Warped.kicad_pcb (KiCad board)
At the start: 2 copper layers, 112 x 90.5 mm, 307 parts, among them J1 USB_C_Receptacle_USB2.0, J2 Conn_01x06_MountingPin, U1 USBLC6-2P6

Commit message: Fix Percent Studio Mod version design
Connections:
- REF** pad 1: (no net) -> GND (x100)
