File: u3-daughterboard/u3-daughterboard.kicad_sch (KiCad schematic)
At the start: 7 parts, among them J1 USB_C_Receptacle_USB2.0, J2 Conn_01x06_MountingPin, U1 USBLC6-2P6

Commit message: Finish U3 design
Parts:
- added H1: MountingHole, MountingHole:MountingHole_3.2mm_M3, symbol Mechanical:MountingHole
- added H2: MountingHole_Pad, MountingHole:MountingHole_3.2mm_M3_Pad_TopBottom, symbol Mechanical:MountingHole_Pad
- J1: footprint u1:USB_C_Receptacle_HRO_TYPE-C-31-M-12 -> BIOI:USB_C_Receptacle_HRO_TYPE-C-31-M-12
- J2: footprint u1:molex_781710004 -> BIOI:molex_781710004
- R1, R2: footprint Resistor_SMD:R_0603_1608Metric -> Resistor_SMD:R_0402_1005Metric
Connections:
- net D+: now also U1.6 (I/O1); no longer U1.4 (I/O2)
- net D-: now also U1.4 (I/O2); no longer U1.6 (I/O1)
- net DN: now also U1.3 (I/O2); no longer U1.1 (I/O1)
- net DP: now also U1.1 (I/O1); no longer U1.3 (I/O2)
- net Earth: now also H2.1; no longer D1.2 (A), U1.2 (GND)
- net GND: now also D1.2 (A), U1.2 (GND)
Changed lines of the file:
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@@
+    (stroke (width 0) (type default))
+  )
+  (wire (pts (xy 149.86 129.54) (xy 149.86 125.73))
     (stroke (width 0) (type default))
   )
@@
     (stroke (width 0) (type default))
   )
-  (global_label "D+" (shape input) (at 143.51 77.47 270) (fields_autoplaced)
-    (effects (font (size 1.27 1.27) (thickness 0.254) bold) (justify right))
-    (property "Intersheetrefs" "${INTERSHEET_REFS}" (at 143.51 82.9924 90)
-      (effects (font (size 1.27 1.27)) (justify right) hide)
+  (global_label "D+" (shape input) (at 143.51 44.45 90) (fields_autoplaced)
+    (effects (font (size 1.27 1.27) (thickness 0.254) bold) (justify left))
+    (property "Intersheetrefs" "${INTERSHEET_REFS}" (at 143.51 38.2734 90)
+      (effects (font (size 1.27 1.27)) (justify left) hide)
     )
   )
@@
     )
   )
-  (global_label "D-" (shape input) (at 143.51 44.45 90) (fields_autoplaced)
-    (effects (font (size 1.27 1.27) (thickness 0.254) bold) (justify left))
-    (property "Intersheetrefs" "${INTERSHEET_REFS}" (at 143.51 38.9276 90)
-      (effects (font (size 1.27 1.27)) (justify left) hide)
+  (global_label "D-" (shape input) (at 143.51 77.47 270) (fields_autoplaced)
+    (effects (font (size 1.27 1.27) (thickness 0.254) bold) (justify right))
+    (property "Intersheetrefs" "${INTERSHEET_REFS}" (at 143.51 83.6466 90)
+      (effects (font (size 1.27 1.27)) (justify right) hide)
     )
   )
@@
     )
   )
-  (global_label "DP" (shape input) (at 138.43 77.47 270) (fields_autoplaced)
+  (global_label "DP" (shape input) (at 138.43 44.45 90) (fields_autoplaced)
+    (effects (font (size 1.27 1.27) (thickness 0.254) bold) (justify left))
+    (property "Intersheetrefs" "${INTERSHEET_REFS}" (at 138.43 38.5758 90)
+      (effects (font (size 1.27 1.27)) (justify left) hide)
+    )
+  )
+  (global_label "DN" (shape input) (at 138.43 77.47 270) (fields_autoplaced)
     (effects (font (size 1.27 1.27) (thickness 0.254) bold) (justify right))
-    (property "Intersheetrefs" "${INTERSHEET_REFS}" (at 138.43 82.69 90)
+    (property "Intersheetrefs" "${INTERSHEET_REFS}" (at 138.43 83.4047 90)
       (effects (font (size 1.27 1.27)) (justify right) hide)
-    )
-  )
-  (global_label "DN" (shape input) (at 138.43 44.45 90) (fields_autoplaced)
-    (effects (font (size 1.27 1.27) (thickness 0.254) bold) (justify left))
-    (property "Intersheetrefs" "${INTERSHEET_REFS}" (at 138.43 39.1695 90)
-      (effects (font (size 1.27 1.27)) (justify left) hide)
     )
   )
@@
       (effects (font (size 1.27 1.27)))
     )
-    (property "Footprint" "u1:USB_C_Receptacle_HRO_TYPE-C-31-M-12" (at 57.15 55.88 0)
+    (property "Footprint" "BIOI:USB_C_Receptacle_HRO_TYPE-C-31-M-12" (at 57.15 55.88 0)
       (effects (font (size 1.27 1.27)) hide)
     )
@@
     )
   )
-  (symbol (lib_id "power:Earth") (at 120.65 59.69 270) (unit 1)
+  (symbol (lib_id "power:Earth") (at 149.86 129.54 0) (unit 1)
     (in_bom yes) (on_board yes) (dnp no) (fields_autoplaced)
-    (property "Reference" "#PWR09" (at 114.3 59.69 0)
-      (effects (font (size 1.27 1.27)) hide)
-    )
-    (property "Value" "Earth" (at 116.84 59.69 0)
-      (effects (font (size 1.27 1.27)) hide)
-    )
-    (property "Footprint" "" (at 120.65 59.69 0)
-      (effects (font (size 1.27 1.27)) hide)
-    )
-    (property "Datasheet" "~" (at 120.65 59.69 0)
-      (effects (font (size 1.27 1.27)) hide)
-    )
-    (pin "1")
-    (instances
-      (project "u3-daughterboard"
-        (path "/2add4f27-2b4b-45f3-834d-7b8d4f9d5b15"
-          (reference "#PWR09") (unit 1)
+    (property "Reference" "#PWR010" (at 149.86 135.89 0)
+      (effects (font (size 1.27 1.27)) hide)
+    )
+    (property "Value" "Earth" (at 149.86 133.35 0)
+      (effects (font (size 1.27 1.27)) hide)
+    )
+    (property "Footprint" "" (at 149.86 129.54 0)
+      (effects (font (size 1.27 1.27)) hide)
+    )
+    (property "Datasheet" "~" (at 149.86 129.54 0)
+      (effects (font (size 1.27 1.27)) hide)
+    )
+    (pin "1")
+    (instances
+      (project "u3-daughterboard"
+        (path "/2add4f27-2b4b-45f3-834d-7b8d4f9d5b15"
+          (reference "#PWR010") (unit 1)
         )
       )
@@
     )
   )
+  (symbol (lib_id "power:GND") (at 176.53 76.2 0) (unit 1)
+    (in_bom yes) (on_board yes) (dnp no)
+    (property "Reference" "#PWR03" (at 176.53 82.55 0)
+      (effects (font (size 1.27 1.27)) hide)
+    )
+    (property "Value" "GND" (at 176.657 80.5942 0)
+      (effects (font (size 1.27 1.27)))
+    )
+    (property "Footprint" "" (at 176.53 76.2 0)
+      (effects (font (size 1.27 1.27)) hide)
+    )
+    (property "Datasheet" "" (at 176.53 76.2 0)
+      (effects (font (size 1.27 1.27)) hide)
+    )
+    (pin "1")
+    (instances
+      (project "u3-daughterboard"
+        (path "/2add4f27-2b4b-45f3-834d-7b8d4f9d5b15"
+          (reference "#PWR03") (unit 1)
+        )
+      )
+      (project "u1"
+        (path "/72a50811-8fa2-4d04-9a96-8be41dc09bc6"
+          (reference "#PWR04") (unit 1)
+        )
+      )
+    )
+  )
   (symbol (lib_id "Device:R_Small") (at 74.93 48.26 270) (unit 1)
     (in_bom yes) (on_board yes) (dnp no)
@@
       (effects (font (size 1.27 1.27)))
     )
-    (property "Footprint" "Resistor_SMD:R_0603_1608Metric" (at 74.93 48.26 0)
+    (property "Footprint" "Resistor_SMD:R_0402_1005Metric" (at 74.93 48.26 0)
       (effects (font (size 1.27 1.27)) hide)
     )
@@
         (path "/72a50811-8fa2-4d04-9a96-8be41dc09bc6"
           (reference "R2") (unit 1)
+        )
+      )
+    )
+  )
+  (symbol (lib_id "Mechanical:MountingHole_Pad") (at 149.86 123.19 0) (unit 1)
+    (in_bom yes) (on_board yes) (dnp no) (fields_autoplaced)
+    (property "Reference" "H2" (at 152.4 120.65 0)
+      (effects (font (size 1.27 1.27)) (justify left))
+    )
+    (property "Value" "MountingHole_Pad" (at 152.4 123.19 0)
+      (effects (font (size 1.27 1.27)) (justify left))
+    )
+    (property "Footprint" "MountingHole:MountingHole_3.2mm_M3_Pad_TopBottom" (at 149.86 123.19 0)
+      (effects (font (size 1.27 1.27)) hide)
+    )
+    (property "Datasheet" "~" (at 149.86 123.19 0)
+      (effects (font (size 1.27 1.27)) hide)
+    )
+    (pin "1")
+    (instances
+      (project "u3-daughterboard"
+        (path "/2add4f27-2b4b-45f3-834d-7b8d4f9d5b15"
+          (reference "H2") (unit 1)
         )
       )
@@
       (effects (font (size 1.27 1.27)) (justify left))
     )
-    (property "Footprint" "u1:molex_781710004" (at 214.63 58.42 0)
+    (property "Footprint" "BIOI:molex_781710004" (at 214.63 58.42 0)
       (effects (font (size 1.27 1.27)) hide)
     )
@@
       (effects (font (size 1.27 1.27)))
     )
-    (property "Footprint" "Resistor_SMD:R_0603_1608Metric" (at 74.93 45.72 0)
+    (property "Footprint" "Resistor_SMD:R_0402_1005Metric" (at 74.93 45.72 0)
       (effects (font (size 1.27 1.27)) hide)
     )
@@
     )
   )
+  (symbol (lib_id "Mechanical:MountingHole") (at 127 121.92 0) (unit 1)
+    (in_bom yes) (on_board yes) (dnp no) (fields_autoplaced)
+    (property "Reference" "H1" (at 129.54 120.65 0)
+      (effects (font (size 1.27 1.27)) (justify left))
+    )
+    (property "Value" "MountingHole" (at 129.54 123.19 0)
+      (effects (font (size 1.27 1.27)) (justify left))
+    )
+    (property "Footprint" "MountingHole:MountingHole_3.2mm_M3" (at 127 121.92 0)
+      (effects (font (size 1.27 1.27)) hide)
+    )
+    (property "Datasheet" "~" (at 127 121.92 0)
+      (effects (font (size 1.27 1.27)) hide)
+    )
+    (instances
+      (project "u3-daughterboard"
+        (path "/2add4f27-2b4b-45f3-834d-7b8d4f9d5b15"
+          (reference "H1") (unit 1)
+        )
+      )
+    )
+  )
   (symbol (lib_id "Device:R_Small") (at 99.06 95.25 0) (unit 1)
     (in_bom yes) (on_board yes) (dnp no)
@@
         (path "/72a50811-8fa2-4d04-9a96-8be41dc09bc6"
           (reference "R2") (unit 1)
-        )
-      )
-    )
-  )
-  (symbol (lib_id "power:Earth") (at 176.53 76.2 0) (unit 1)
-    (in_bom yes) (on_board yes) (dnp no) (fields_autoplaced)
-    (property "Reference" "#PWR03" (at 176.53 82.55 0)
-      (effects (font (size 1.27 1.27)) hide)
-    )
-    (property "Value" "Earth" (at 176.53 80.01 0)
-      (effects (font (size 1.27 1.27)) hide)
-    )
-    (property "Footprint" "" (at 176.53 76.2 0)
-      (effects (font (size 1.27 1.27)) hide)
-    )
-    (property "Datasheet" "~" (at 176.53 76.2 0)
-      (effects (font (size 1.27 1.27)) hide)
-    )
-    (pin "1")
-    (instances
-      (project "u3-daughterboard"
-        (path "/2add4f27-2b4b-45f3-834d-7b8d4f9d5b15"
-          (reference "#PWR03") (unit 1)
         )
       )
@@
         )
       )
+    )
+  )
+  (symbol (lib_id "power:GND") (at 120.65 59.69 270) (unit 1)
+    (in_bom yes) (on_board yes) (dnp no)
+    (property "Reference" "#PWR09" (at 114.3 59.69 0)
+      (effects (font (size 1.27 1.27)) hide)
+    )
+    (property "Value" "GND" (at 116.2558 59.817 0)
+      (effects (font (size 1.27 1.27)))
+    )
+    (property "Footprint" "" (at 120.65 59.69 0)
+      (effects (font (size 1.27 1.27)) hide)
+    )
+    (property "Datasheet" "" (at 120.65 59.69 0)
+      (effects (font (size 1.27 1.27)) hide)
+    )
+    (pin "1")
+    (instances
+      (project "u3-daughterboard"
+        (path "/2add4f27-2b4b-45f3-834d-7b8d4f9d5b15"
+          (reference "#PWR09") (unit 1)
+        )
+      )
+      (project "u1"
+        (path "/72a50811-8fa2-4d04-9a96-8be41dc09bc6"
+          (reference "#PWR04") (unit 1)
+        )
+      )

Commit message: Finish U3 daughterboard production files
Parts:
- added C1: 100nF, Capacitor_SMD:C_0402_1005Metric, symbol Device:C_Small
Connections:
- net GND: now also C1.2
- net UVCC: now also C1.1
Changed lines of the file:
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@@
+    (stroke (width 0) (type default))
+  )
+  (wire (pts (xy 114.3 97.79) (xy 114.3 102.87))
     (stroke (width 0) (type default))
   )
@@
   )
   (wire (pts (xy 68.58 55.88) (xy 68.58 53.34))
+    (stroke (width 0) (type default))
+  )
+  (wire (pts (xy 114.3 87.63) (xy 114.3 92.71))
     (stroke (width 0) (type default))
   )
@@
     (effects (font (size 1.27 1.27) (thickness 0.254) bold) (justify left))
     (property "Intersheetrefs" "${INTERSHEET_REFS}" (at 176.53 46.3167 90)
+      (effects (font (size 1.27 1.27)) (justify left) hide)
+    )
+  )
+  (global_label "UVCC" (shape input) (at 114.3 87.63 90) (fields_autoplaced)
+    (effects (font (size 1.27 1.27) (thickness 0.254) bold) (justify left))
+    (property "Intersheetrefs" "${INTERSHEET_REFS}" (at 114.3 79.3367 90)
       (effects (font (size 1.27 1.27)) (justify left) hide)
     )
@@
     )
   )
+  (symbol (lib_id "power:GND") (at 114.3 102.87 0) (unit 1)
+    (in_bom yes) (on_board yes) (dnp no)
+    (property "Reference" "#PWR011" (at 114.3 109.22 0)
+      (effects (font (size 1.27 1.27)) hide)
+    )
+    (property "Value" "GND" (at 114.427 107.2642 0)
+      (effects (font (size 1.27 1.27)))
+    )
+    (property "Footprint" "" (at 114.3 102.87 0)
+      (effects (font (size 1.27 1.27)) hide)
+    )
+    (property "Datasheet" "" (at 114.3 102.87 0)
+      (effects (font (size 1.27 1.27)) hide)
+    )
+    (pin "1")
+    (instances
+      (project "u3-daughterboard"
+        (path "/2add4f27-2b4b-45f3-834d-7b8d4f9d5b15"
+          (reference "#PWR011") (unit 1)
+        )
+      )
+      (project "u1"
+        (path "/72a50811-8fa2-4d04-9a96-8be41dc09bc6"
+          (reference "#PWR04") (unit 1)
+        )
+      )
+    )
+  )
   (symbol (lib_id "power:GND") (at 176.53 76.2 0) (unit 1)
     (in_bom yes) (on_board yes) (dnp no)
@@
         )
       )
+    )
+  )
+  (symbol (lib_id "Device:C_Small") (at 114.3 95.25 0) (unit 1)
+    (in_bom yes) (on_board yes) (dnp no) (fields_autoplaced)
+    (property "Reference" "C1" (at 116.84 93.9863 0)
+      (effects (font (size 1.27 1.27)) (justify left))
+    )
+    (property "Value" "100nF" (at 116.84 96.5263 0)
+      (effects (font (size 1.27 1.27)) (justify left))
+    )
+    (property "Footprint" "Capacitor_SMD:C_0402_1005Metric" (at 114.3 95.25 0)
+      (effects (font (size 1.27 1.27)) hide)
+    )
+    (property "Datasheet" "~" (at 114.3 95.25 0)
+      (effects (font (size 1.27 1.27)) hide)
+    )
+    (pin "1")
+    (pin "2")
+    (instances
+      (project "u3-daughterboard"
+        (path "/2add4f27-2b4b-45f3-834d-7b8d4f9d5b15"
+          (reference "C1") (unit 1)
+        )
+      )
