File: without-power-switch/u1.kicad_pcb (KiCad board)
At the start: 2 copper layers, 18 x 16.5 mm, 12 parts, among them J1 USB_C_Receptacle_USB2.0, J2 Conn_01x06_MountingPin, U1 USBLC6-2P6

Commit message: Add rendering files
Other:
- net class Default removed

Commit message: Update U1 panelized production files
Parts:
- removed the REF** at (63.0, 43.2)
- removed the REF** at (45.0, 43.2)
Connections:
- REF** pad 1: (no net) -> GND (x4)

Commit message: Add new U1 panelized production files
Other:
- board text added: "G+-V"
