File: without-power-switch-using-fpc-connector/u1.kicad_pcb (KiCad board)
At the start: 2 copper layers, 18 x 16.5 mm, 10 parts, among them J1 USB_C_Receptacle_USB2.0, J2 Conn_01x06_MountingPin, U1 USBLC6-2P6

Commit message: Update model of U1 with FPC connector
Parts:
- added REF**: Mouse_Bite_7, u1:Mouse_Bite_7, F.Cu at (63.0, 43.2)
- added REF**: Mouse_Bite_7, u1:Mouse_Bite_7, F.Cu at (45.0, 43.2)
